File: kicadFiles/tsuki.kicad_pcb (KiCad board)
At the start: 2 copper layers, 283 x 94.2 mm, 227 parts, among them J1 TYPE-C-31-M12_13, J2 Conn_01x14, J3 Conn_ARM_JTAG_SWD_10, Q1 BSS138, SW1 ESC, SW10 9, SW11 0, SW12 -_, SW13 +=, SW14 2U BKSP, SW15 TAB_150, SW16 Q, SW17 W, SW18 E, SW19 R, SW2 1, SW20 T, SW21 Y, SW22 U, SW23 I, SW24 O, SW25 P, SW26 [{, SW27 ]}, SW28 \|_150, SW29 CAPS_175, SW3 2, SW30 A, SW31 S, SW32 D, SW33 F, SW34 G, SW35 H, SW36 J, SW37 K, SW38 L, SW39 :;, SW4 3, SW40 "', SW41 ENTER_225, SW42 LSHIFT_225, SW43 Z, SW44 X, SW45 C, SW46 V, SW47 B, SW48 N, SW49 M, SW5 4, SW50 <,, SW51 >., SW52 ?/, SW53 RSHIFT_275, SW54 LCTRL_150, SW55 LGUI_100, SW56 LALT_150, SW58 RALT_150, SW59 RGUI_150, SW6 5, SW60 RCTRL_150, SW61 FN_100, SW62 RSHIFT_175, SW63 STEPPED_CAPS_125, SW64 1U LBKSP, SW65 1U RBKSP, SW66 ISO_100, SW67 ISO_ENTER, SW68 LCTRL_125, SW69 LGUI_125, SW7 6, SW70 LGUI_100, SW71 LALT_125, SW72 LALT_150, SW75 SPACE_625, SW77 SPACE_700, SW8 7, SW80 RALT_125, SW81 RALT_150, SW83 RGUI_125, SW84 RGUI_100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

Commit message: Added bottom row documentation
Parts:
- added L5: Warning, acheron_Graphics:warning_sign_3.6x3.2mm, F.Cu at (81.0, 144.2)
- added L6: Warning, acheron_Graphics:warning_sign_3.6x3.2mm, F.Cu at (80.9, 84.9)
- added L7: Warning, acheron_Graphics:warning_sign_3.6x3.2mm, F.Cu at (99.3, 120.7)
- added L8: Warning, acheron_Graphics:warning_sign_3.6x3.2mm, F.Cu at (318.0, 139.4)
- added L9: Warning, acheron_Graphics:warning_sign_3.6x3.2mm, F.Cu at (112.1, 139.9)
- added LED1: LED, acheron_Components:LED_THT_2.54mm, F.Cu at (346.2, 96.4)
- added LED10: LED, acheron_Components:LED_THT_2.54mm, F.Cu at (174.7, 96.4)
- added LED11: LED, acheron_Components:LED_THT_2.54mm, F.Cu at (155.7, 96.4)
- added LED12: LED, acheron_Components:LED_THT_2.54mm, F.Cu at (136.6, 96.4)
- added LED13: LED, acheron_Components:LED_THT_2.54mm, F.Cu at (117.6, 96.4)
- added LED14: LED, acheron_Components:LED_THT_2.54mm, F.Cu at (98.5, 96.4)
- added LED15: LED, acheron_Components:LED_THT_2.54mm, F.Cu at (89.0, 96.4)
- added LED16: LED, acheron_Components:LED_THT_2.54mm, F.Cu at (79.5, 96.4)
- added LED17: LED, acheron_Components:LED_THT_2.54mm, F.Cu at (341.4, 115.5)
- added LED18: LED, acheron_Components:LED_THT_2.54mm, F.Cu at (317.6, 115.5)
- added LED19: LED, acheron_Components:LED_THT_2.54mm, F.Cu at (298.6, 115.5)
- added LED2: LED, acheron_Components:LED_THT_2.54mm, F.Cu at (327.1, 96.4)
- added LED20: LED, acheron_Components:LED_THT_2.54mm, F.Cu at (279.5, 115.5)
- added LED21: LED, acheron_Components:LED_THT_2.54mm, F.Cu at (260.5, 115.5)
- added LED22: LED, acheron_Components:LED_THT_2.54mm, F.Cu at (241.4, 115.5)
- added LED23: LED, acheron_Components:LED_THT_2.54mm, F.Cu at (222.4, 115.5)
- added LED24: LED, acheron_Components:LED_THT_2.54mm, F.Cu at (203.3, 115.5)
- added LED25: LED, acheron_Components:LED_THT_2.54mm, F.Cu at (184.3, 115.5)
- added LED26: LED, acheron_Components:LED_THT_2.54mm, F.Cu at (165.2, 115.5)
- added LED27: LED, acheron_Components:LED_THT_2.54mm, F.Cu at (146.2, 115.5)
- added LED28: LED, acheron_Components:LED_THT_2.54mm, F.Cu at (127.1, 115.5)
- added LED29: LED, acheron_Components:LED_THT_2.54mm, F.Cu at (108.1, 115.5)
- added LED3: LED, acheron_Components:LED_THT_2.54mm, F.Cu at (308.1, 96.4)
- added LED30: LED, acheron_Components:LED_THT_2.54mm, F.Cu at (444.4, 112.7)
- added LED31: LED, acheron_Components:LED_THT_2.54mm, F.Cu at (84.2, 115.5)
- added LED32: LED, acheron_Components:LED_THT_2.54mm, F.Cu at (437.1, 122.1)
- added LED4: LED, acheron_Components:LED_THT_2.54mm, F.Cu at (289.0, 96.4)
- added LED5: LED, acheron_Components:LED_THT_2.54mm, F.Cu at (270.0, 96.4)
- added LED6: LED, acheron_Components:LED_THT_2.54mm, F.Cu at (250.9, 96.4)
- added LED7: LED, acheron_Components:LED_THT_2.54mm, F.Cu at (231.9, 96.4)
- added LED8: LED, acheron_Components:LED_THT_2.54mm, F.Cu at (212.8, 96.4)
- added LED9: LED, acheron_Components:LED_THT_2.54mm, F.Cu at (193.8, 96.4)
- added Q2: AO4407A, acheron_Components:SOIC-8, F.Cu at (399.0, 143.6)
- added QRST2: DTC123J, Package_TO_SOT_SMD:SOT-23, F.Cu at (411.4, 141.6)
- added RL1: 420R, acheron_Components:R_SMD_1206, F.Cu at (350.0, 95.4)
- added RL10: 420R, acheron_Components:R_SMD_1206, F.Cu at (169.4, 95.2)
- added RL11: 420R, acheron_Components:R_SMD_1206, F.Cu at (150.9, 96.4)
- added RL12: 420R, acheron_Components:R_SMD_1206, F.Cu at (131.0, 96.2)
- added RL13: 420R, acheron_Components:R_SMD_1206, F.Cu at (111.7, 95.2)
- added RL14: 420R, acheron_Components:R_SMD_1206, F.Cu at (93.7, 95.7)
- added RL16: 420R, acheron_Components:R_SMD_1206, F.Cu at (73.8, 95.3)
- added RL17: 420R, acheron_Components:R_SMD_1206, F.Cu at (416.2, 110.2)
- added RL18: 420R, acheron_Components:R_SMD_1206, F.Cu at (422.1, 106.9)
- added RL19: 420R, acheron_Components:R_SMD_1206, F.Cu at (416.2, 113.5)
- added RL2: 420R, acheron_Components:R_SMD_1206, F.Cu at (321.8, 95.7)
- added RL20: 420R, acheron_Components:R_SMD_1206, F.Cu at (422.1, 110.2)
- added RL21: 420R, acheron_Components:R_SMD_1206, F.Cu at (428.1, 106.9)
- added RL22: 420R, acheron_Components:R_SMD_1206, F.Cu at (416.2, 116.8)
- added RL23: 420R, acheron_Components:R_SMD_1206, F.Cu at (422.1, 113.5)
- added RL24: 420R, acheron_Components:R_SMD_1206, F.Cu at (428.1, 110.2)
- added RL25: 420R, acheron_Components:R_SMD_1206, F.Cu at (416.2, 120.1)
- added RL26: 420R, acheron_Components:R_SMD_1206, F.Cu at (434.0, 106.9)
- added RL27: 420R, acheron_Components:R_SMD_1206, F.Cu at (422.1, 116.8)
- added RL28: 420R, acheron_Components:R_SMD_1206, F.Cu at (428.1, 113.5)
- added RL29: 420R, acheron_Components:R_SMD_1206, F.Cu at (434.0, 110.2)
- added RL3: 420R, acheron_Components:R_SMD_1206, F.Cu at (301.5, 95.2)
- added RL30: 420R, acheron_Components:R_SMD_1206, F.Cu at (422.1, 120.1)
- added RL31: 420R, acheron_Components:R_SMD_1206, F.Cu at (440.0, 106.9)
- added RL32: 420R, acheron_Components:R_SMD_1206, F.Cu at (416.2, 106.9)
- added RL4: 420R, acheron_Components:R_SMD_1206, F.Cu at (283.9, 96.2)
- added RL5: 420R, acheron_Components:R_SMD_1206, F.Cu at (264.9, 95.2)
- added RL6: 420R, acheron_Components:R_SMD_1206, F.Cu at (245.8, 95.4)
- added RL7: 420R, acheron_Components:R_SMD_1206, F.Cu at (226.8, 95.4)
- added RL8: 420R, acheron_Components:R_SMD_1206, F.Cu at (206.7, 95.2)
- added RL9: 420R, acheron_Components:R_SMD_1206, F.Cu at (188.4, 95.2)
- added RLED1: 10k, acheron_Components:R_SMD_1206, F.Cu at (406.2, 141.0)
- added RLED2: 100R, acheron_Components:R_SMD_1206, F.Cu at (403.6, 148.5)
- added RLED3: 10k, acheron_Components:R_SMD_1206, F.Cu at (406.2, 144.3)
- L1: moved to F.Cu
- L4: moved to B.Cu
- SW67: footprint acheron_MX_SolderMask:MX_ISOEnter_Vertical -> acheron_MX_SolderMask:MX_ISOEnter_Vertical_LED
- moved L1 59.5 mm to (248.9, 167.3), turned to 0 degrees
- moved RSI1 58.9 mm to (397.3, 99.7)
- moved RSO1 58.9 mm to (397.3, 103.0)
- moved U3 58.9 mm to (398.6, 103.3)
- moved CRST1 58.9 mm to (399.6, 100.9)
- moved CSO1 58.9 mm to (396.2, 98.5)
- moved L4 20.8 mm to (249.0, 167.2), turned to 180 degrees
- moved DF1 11.2 mm to (336.2, 103.1)
- moved F1 11.2 mm to (332.8, 103.0)
- moved D1 9.62 mm to (347.4, 85.4)
- moved D9 5.00 mm to (198.5, 96.4)
- moved D10 4.99 mm to (179.5, 96.4)
- moved D4 4.69 mm to (294.1, 96.4)
- moved D7 4.45 mm to (237.2, 96.4)
- moved D11 3.59 mm to (161.6, 95.2)
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Connections:
- SW55 pad 1: Col2 -> L2
- SW55 pad 2: L2 -> Col2
- SW63 pad 1: Col1 -> Net-(D29-Pad2)
- SW63 pad 2: Net-(D29-Pad2) -> Col1
Other:
- board text added: "(H) 1U LGUI"
- board text added: "(H,T) 1.50U LCTRL"
- board text added: "(T) 1U LGUI"
- board text added: "1.25U LCTRL (D)"
- board text added: "1.25U LGUI (D)"
- board text added: "1.50U RGUI (H)"
- board text added: "6.0/6.25U STAB"
- board text added: "6.0/7.0U STAB"
- board text added: "6.25U STAB"
- board text added: "7U STAB"
- board text added: "ANSI ENTER"
- board text added: "ISO ENTER"
- board text added: "ISO ~~#"
- board text added: "STEPPED"
- board text removed: "(H) 1.50U RGUI"
- board text removed: "1.25U LCTRL"
- board text removed: "1.25U LGUI"
- board text removed: "1.50U LCTRL"
- board text removed: "1U LGUI"

Commit message: Routed second row LEDs
Parts:
- removed D60: 1N4148, acheron_Components:D_SOD-123
- added LED33: LED, acheron_Components:LED_THT_2.54mm, F.Cu at (293.8, 134.5)
- added LED34: LED, acheron_Components:LED_THT_2.54mm, F.Cu at (274.7, 134.5)
- added LED35: LED, acheron_Components:LED_THT_2.54mm, F.Cu at (255.7, 134.5)
- added LED36: LED, acheron_Components:LED_THT_2.54mm, F.Cu at (236.6, 134.5)
- added LED37: LED, acheron_Components:LED_THT_2.54mm, F.Cu at (217.6, 134.5)
- added LED38: LED, acheron_Components:LED_THT_2.54mm, F.Cu at (198.5, 134.5)
- added LED39: LED, acheron_Components:LED_THT_2.54mm, F.Cu at (179.5, 134.5)
- added LED40: LED, acheron_Components:LED_THT_2.54mm, F.Cu at (160.4, 134.5)
- added LED41: LED, acheron_Components:LED_THT_2.54mm, F.Cu at (141.4, 134.5)
- added LED42: LED, acheron_Components:LED_THT_2.54mm, F.Cu at (122.3, 134.5)
- added LED43: LED, acheron_Components:LED_THT_2.54mm, F.Cu at (103.3, 134.5)
- added LED44: LED, acheron_Components:LED_THT_2.54mm, F.Cu at (91.4, 134.5)
- added LED45: LED, acheron_Components:LED_THT_2.54mm, F.Cu at (193.7, 55.8)
- added LED46: LED, acheron_Components:LED_THT_2.54mm, F.Cu at (199.6, 52.5)
- added LED47: LED, acheron_Components:LED_THT_2.54mm, F.Cu at (193.7, 58.6)
- added LED48: LED, acheron_Components:LED_THT_2.54mm, F.Cu at (192.4, 61.9)
- added RGND1: R01, acheron_Components:R_SMD_1206, F.Cu at (368.5, 153.8)
- added RL15: 420R, acheron_Components:R_SMD_1206, F.Cu at (171.5, 50.0)
- added RL33: 420R, acheron_Components:R_SMD_1206, F.Cu at (177.4, 46.7)
- added RL34: 420R, acheron_Components:R_SMD_1206, F.Cu at (171.5, 53.3)
- added RL35: 420R, acheron_Components:R_SMD_1206, F.Cu at (177.4, 50.0)
- added RL36: 420R, acheron_Components:R_SMD_1206, F.Cu at (183.4, 46.7)
- added RL37: 420R, acheron_Components:R_SMD_1206, F.Cu at (171.5, 56.6)
- added RL38: 420R, acheron_Components:R_SMD_1206, F.Cu at (177.4, 53.3)
- added RL39: 420R, acheron_Components:R_SMD_1206, F.Cu at (183.4, 50.0)
- added RL40: 420R, acheron_Components:R_SMD_1206, F.Cu at (171.5, 59.9)
- added RL41: 420R, acheron_Components:R_SMD_1206, F.Cu at (189.3, 46.7)
- added RL42: 420R, acheron_Components:R_SMD_1206, F.Cu at (177.4, 56.6)
- added RL43: 420R, acheron_Components:R_SMD_1206, F.Cu at (183.4, 53.3)
- added RL44: 420R, acheron_Components:R_SMD_1206, F.Cu at (189.3, 50.0)
- added RL45: 420R, acheron_Components:R_SMD_1206, F.Cu at (177.4, 59.9)
- added RL46: 420R, acheron_Components:R_SMD_1206, F.Cu at (195.3, 46.7)
- added RL47: 420R, acheron_Components:R_SMD_1206, F.Cu at (171.5, 46.7)
- moved LED30 360.1 mm to (84.2, 115.5)
- moved RL30 346.3 mm to (75.9, 112.8), turned to 90 degrees
- moved RL29 330.8 mm to (103.3, 114.0), turned to 90 degrees
- moved RL28 305.8 mm to (122.3, 114.0), turned to 90 degrees
- moved RL27 280.8 mm to (141.4, 114.0), turned to 90 degrees
- moved RL26 273.7 mm to (160.4, 114.0), turned to 90 degrees
- moved RL25 236.8 mm to (179.5, 114.0), turned to 90 degrees
- moved RL24 229.6 mm to (198.5, 114.0), turned to 90 degrees
- moved SW66 219.9 mm to (322.4, 148.5)
- moved SW88 219.9 mm to (103.3, 129.5)
- moved D67 219.2 mm to (108.1, 133.0), turned to 90 degrees
- moved D61 215.1 mm to (327.1, 152.1)
- moved RL23 204.6 mm to (217.6, 114.0), turned to 90 degrees
- moved RL22 179.6 mm to (236.6, 114.0), turned to 90 degrees
- moved RL21 172.6 mm to (255.7, 114.0), turned to 90 degrees
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Connections:
- CB1 pad 1: GND -> GNDD
- CB2 pad 1: GND -> GNDD
- CB3 pad 1: GND -> GNDD
- CB4 pad 1: GND -> GNDD
- CB5 pad 1: GND -> GNDD
- CB6 pad 1: GND -> GNDD
- CB7 pad 2: GND -> GNDD
- CB8 pad 1: GND -> GNDD
- RGUI_125 pad 1: Col10 -> Col12
- SW28 pad 1: Col14 -> Col13
- SW41 pad 1: Col13 -> Col14
- SW58 pad 1: Col10 -> Col12
- SW59 pad 2: Col11 -> Col13
- SW60 pad 1: Col12 -> Col14
- SW67 pad 1: Col13 -> Col14
- SW81 pad 1: Col10 -> Col12
- SW83 pad 1: Col11 -> Col13
- SW84 pad 1: Col11 -> Col13
- SW86 pad 1: Col12 -> Col14
- U1 pad 10: Col7 -> Net-(U1-Pad10)
- U1 pad 11: Col6 -> Net-(U1-Pad11)
- U1 pad 12: Col5 -> Net-(U1-Pad12)
- U1 pad 13: Col4 -> Net-(U1-Pad13)
- U1 pad 14: Col3 -> Net-(U1-Pad14)
- U1 pad 15: Col2 -> Net-(U1-Pad15)
- U1 pad 16: Row3 -> Net-(U1-Pad16)
- U1 pad 17: Row4 -> Net-(U1-Pad17)
- U1 pad 18: Col1 -> Net-(U1-Pad18)
- U1 pad 19: Row5 -> Net-(U1-Pad19)
- U1 pad 2: Col12 -> Net-(U1-Pad2)
- U1 pad 20: Extra14 -> Net-(U1-Pad20)
- U1 pad 21: Extra13 -> Net-(U1-Pad21)
- U1 pad 22: Extra12 -> Net-(U1-Pad22)
- U1 pad 23: GND -> GNDD
- U1 pad 25: Extra11 -> Col1
- U1 pad 26: Extra10 -> Net-(U1-Pad26)
- U1 pad 27: Extra9 -> Net-(U1-Pad27)
- U1 pad 28: Extra8 -> Net-(U1-Pad28)
- U1 pad 29: Extra7 -> Net-(U1-Pad29)
- U1 pad 3: Col11 -> Net-(U1-Pad3)
- U1 pad 30: Extra6 -> Net-(U1-Pad30)
- U1 pad 31: Extra5 -> Net-(U1-Pad31)
- U1 pad 35: GND -> GNDD
- U1 pad 38: Extra4 -> Net-(U1-Pad38)
- U1 pad 39: Extra3 -> Net-(U1-Pad39)
- U1 pad 4: Col10 -> Net-(U1-Pad4)
- U1 pad 40: Extra2 -> Net-(U1-Pad40)
- U1 pad 41: RGB_3V3 -> Net-(U1-Pad41)
- U1 pad 42: Row2 -> Net-(U1-Pad42)
- U1 pad 43: Row1 -> Net-(U1-Pad43)
- U1 pad 45: Col14 -> Net-(U1-Pad45)
- U1 pad 46: Col13 -> Net-(U1-Pad46)
- U1 pad 47: GND -> GNDD
- U1 pad 5: Col9 -> Net-(U1-Pad5)
- U1 pad 6: Col8 -> Net-(U1-Pad6)
- U1 pad 8: GND -> GNDD
Routing:
- net Net-(Q2-Pad1): track 0.00 -> 552.3 mm
- net 3.3V: track 0.00 -> 317.7 mm, vias 0 -> 7
- net NRST: track 0.00 -> 294.4 mm, vias 0 -> 1
- net Row2: track 0.00 -> 281.2 mm
- net SWCLK: track 0.00 -> 274.8 mm, vias 0 -> 1
- net Net-(U1-Pad13): track 0.00 -> 268.5 mm
- net Row3: track 0.00 -> 267.1 mm
- net Row1: track 0.00 -> 266.0 mm
- net SWDIO: track 0.00 -> 260.5 mm, vias 0 -> 1
- net Net-(U1-Pad14): track 0.00 -> 250.5 mm
- net Net-(U1-Pad15): track 0.00 -> 241.3 mm
- net BOOT0: track 0.00 -> 239.2 mm, vias 0 -> 2
- net Net-(U1-Pad16): track 0.00 -> 205.8 mm
- net Net-(U1-Pad17): track 0.00 -> 187.5 mm
- net Col13: track 0.00 -> 179.2 mm
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- added copper zone on B.Cu, net (none)
- added copper zone on B.Cu, net 3.3V
- added copper zone on F.Cu, net GNDD
Other:
- net class DiffPair: clearance 0.508 -> 0.1524
- rule via_min_size: 0.508 -> 0.4572
