File: kicadFiles/tsuki.kicad_pcb (KiCad board)
At the start: 2 copper layers, 283 x 94.2 mm, 332 parts, among them J1 TYPE-C-31-M12_13, J2 Conn_01x14, J3 Conn_ARM_JTAG_SWD_10, Q1 BSS138, Q2 AO4407A, SW1 ESC, SW10 9, SW11 0, SW12 -_, SW13 +=, SW14 2U BKSP, SW15 TAB_150, SW16 Q, SW17 W, SW18 E, SW19 R, SW2 1, SW20 T, SW21 Y, SW22 U, SW23 I, SW24 O, SW25 P, SW26 [{, SW27 ]}, SW28 \|_150, SW29 CAPS_175, SW3 2, SW30 A, SW31 S, SW32 D, SW33 F, SW34 G, SW35 H, SW36 J, SW37 K, SW38 L, SW39 :;, SW4 3, SW40 "', SW41 ENTER_225, SW42 LSHIFT_225, SW43 Z, SW44 X, SW45 C, SW46 V, SW47 B, SW48 N, SW49 M, SW5 4, SW50 <,, SW51 >., SW52 ?/, SW53 RSHIFT_275, SW54 LCTRL_150, SW55 LGUI_100, SW56 LALT_150, SW58 RALT_150, SW59 RGUI_150, SW6 5, SW60 RCTRL_150, SW61 FN_100, SW62 RSHIFT_175, SW63 STEPPED_CAPS_125, SW64 1U LBKSP, SW65 1U RBKSP, SW66 ISO_100, SW67 ISO_ENTER, SW68 LCTRL_125, SW69 LGUI_125, SW7 6, SW70 LGUI_100, SW71 LALT_125, SW72 LALT_150, SW75 SPACE_625, SW77 SPACE_700, SW8 7, SW80 RALT_125, SW81 RALT_150, SW83 RGUI_125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

Commit message: Finished routing
Parts:
- removed RL47: 420R, acheron_Components:R_SMD_1206
- removed SW48: N, acheron_MX_SolderMask:MX100
- added L10: Tsuki Big Logo, tsukiGraphics:tsukiLogo_90x115mm, B.Cu at (145.0, 129.5)
- added LED49: LED, acheron_Components:LED_THT_2.54mm, F.Cu at (322.4, 153.6)
- added LED50: LED, acheron_Components:LED_THT_2.54mm, F.Cu at (303.3, 153.6)
- added LED51: LED, acheron_Components:LED_THT_2.54mm, F.Cu at (284.3, 153.6)
- added LED52: LED, acheron_Components:LED_THT_2.54mm, F.Cu at (265.2, 153.6)
- added LED53: LED, acheron_Components:LED_THT_2.54mm, F.Cu at (246.2, 153.6)
- added LED54: LED, acheron_Components:LED_THT_2.54mm, F.Cu at (227.1, 153.6)
- added LED55: LED, acheron_Components:LED_THT_2.54mm, F.Cu at (208.1, 153.6)
- added LED56: LED, acheron_Components:LED_THT_2.54mm, F.Cu at (189.0, 153.6)
- added LED57: LED, acheron_Components:LED_THT_2.54mm, F.Cu at (170.0, 153.6)
- added LED58: LED, acheron_Components:LED_THT_2.54mm, F.Cu at (150.9, 153.6)
- added LED59: LED, acheron_Components:LED_THT_2.54mm, F.Cu at (131.9, 153.6)
- added LED60: LED, acheron_Components:LED_THT_2.54mm, F.Cu at (112.8, 153.6)
- added LED61: LED, acheron_Components:LED_THT_2.54mm, F.Cu at (96.1, 153.6)
- added LED62: LED, acheron_Components:LED_THT_2.54mm, F.Cu at (86.6, 153.6)
- added LED63: LED, acheron_Components:LED_THT_2.54mm, F.Cu at (343.8, 172.6)
- added LED64: LED, acheron_Components:LED_THT_2.54mm, F.Cu at (341.4, 172.6)
- added LED65: LED, acheron_Components:LED_THT_2.54mm, F.Cu at (320.0, 172.6)
- added LED66: LED, acheron_Components:LED_THT_2.54mm, F.Cu at (315.2, 172.6)
- added LED67: LED, acheron_Components:LED_THT_2.54mm, F.Cu at (312.8, 172.6)
- added LED68: LED, acheron_Components:LED_THT_2.54mm, F.Cu at (296.2, 172.6)
- added LED69: LED, acheron_Components:LED_THT_2.54mm, F.Cu at (293.8, 172.6)
- added LED70: LED, acheron_Components:LED_THT_2.54mm, F.Cu at (284.3, 172.6)
- added LED71: LED, acheron_Components:LED_THT_2.54mm, F.Cu at (224.7, 172.6)
- added LED72: LED, acheron_Components:LED_THT_2.54mm, F.Cu at (212.8, 172.6)
- added LED73: LED, acheron_Components:LED_THT_2.54mm, F.Cu at (153.3, 172.6)
- added LED74: LED, acheron_Components:LED_THT_2.54mm, F.Cu at (141.4, 172.6)
- added LED75: LED, acheron_Components:LED_THT_2.54mm, F.Cu at (131.9, 172.6)
- added LED76: LED, acheron_Components:LED_THT_2.54mm, F.Cu at (129.5, 172.6)
- added LED77: LED, acheron_Components:LED_THT_2.54mm, F.Cu at (112.8, 172.6)
- added LED78: LED, acheron_Components:LED_THT_2.54mm, F.Cu at (108.1, 172.6)
- added LED79: LED, acheron_Components:LED_THT_2.54mm, F.Cu at (105.7, 172.6)
- added LED80: LED, acheron_Components:LED_THT_2.54mm, F.Cu at (84.2, 172.6)
- added LED81: LED, acheron_Components:LED_THT_2.54mm, F.Cu at (81.9, 172.6)
- added RL48: 420R, acheron_Components:R_SMD_1206, F.Cu at (298.6, 152.1)
- added RL49: 420R, acheron_Components:R_SMD_1206, F.Cu at (279.5, 152.1)
- added RL50: 420R, acheron_Components:R_SMD_1206, F.Cu at (260.5, 152.1)
- added RL51: 420R, acheron_Components:R_SMD_1206, F.Cu at (241.4, 152.1)
- added RL52: 420R, acheron_Components:R_SMD_1206, F.Cu at (222.4, 152.1)
- added RL53: 420R, acheron_Components:R_SMD_1206, F.Cu at (203.3, 152.1)
- added RL54: 420R, acheron_Components:R_SMD_1206, F.Cu at (184.3, 152.1)
- added RL55: 420R, acheron_Components:R_SMD_1206, F.Cu at (165.2, 152.1)
- added RL56: 420R, acheron_Components:R_SMD_1206, F.Cu at (146.2, 152.1)
- added RL57: 420R, acheron_Components:R_SMD_1206, F.Cu at (127.1, 152.1)
- added RL58: 420R, acheron_Components:R_SMD_1206, F.Cu at (117.6, 152.1)
- added RL60: 420R, acheron_Components:R_SMD_1206, F.Cu at (81.9, 152.1)
- added RL61: 420R, acheron_Components:R_SMD_1206, F.Cu at (336.1, 172.9)
- added RL63: 420R, acheron_Components:R_SMD_1206, F.Cu at (325.3, 172.9)
- added RL66: 420R, acheron_Components:R_SMD_1206, F.Cu at (301.5, 172.9)
- added RL68: 420R, acheron_Components:R_SMD_1206, F.Cu at (279.5, 172.9)
- added RL69: 420R, acheron_Components:R_SMD_1206, F.Cu at (218.8, 172.3)
- added RL71: 420R, acheron_Components:R_SMD_1206, F.Cu at (147.3, 173.5)
- added RL73: 420R, acheron_Components:R_SMD_1206, F.Cu at (123.5, 173.5)
- added RL75: 420R, acheron_Components:R_SMD_1206, F.Cu at (118.2, 173.5)
- added RL77: 420R, acheron_Components:R_SMD_1206, F.Cu at (89.6, 173.5)
- moved CRGB5 369.7 mm to (112.0, 102.0), turned to 270 degrees
- moved RRGB5 354.6 mm to (109.7, 101.3), turned to 270 degrees
- moved CRGB6 346.5 mm to (122.1, 157.0), turned to 270 degrees
- moved RRGB6 345.2 mm to (124.3, 157.8), turned to 90 degrees
- moved CRGB4 316.4 mm to (162.0, 101.3), turned to 270 degrees
- moved CRGB7 304.7 mm to (160.0, 159.0), turned to 270 degrees
- moved RRGB4 299.3 mm to (159.7, 101.0), turned to 270 degrees
- moved RRGB7 297.9 mm to (159.1, 156.0)
- moved LED31 282.5 mm to (343.8, 134.5)
- moved CRGB3 276.2 mm to (207.1, 102.0), turned to 270 degrees
- moved RRGB3 259.6 mm to (204.8, 101.3), turned to 270 degrees
- moved RRGB8 256.1 mm to (207.2, 157.1), turned to 270 degrees
- moved CRGB8 255.6 mm to (209.4, 157.9), turned to 90 degrees
- moved RRGB9 213.7 mm to (256.0, 156.9)
- moved CRGB9 212.3 mm to (256.8, 159.0), turned to 180 degrees
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- renumbered CRST1 to CR1, CRST2 to CR2, DRST1 to DR1, RRST1 to RR1, SWRST1 to SWR1
Connections:
- LED32 pad A: Net-(LED32-PadA) -> Net-(LED31-PadA)
- LED48 pad A: Net-(LED48-PadA) -> Net-(LED47-PadA)
- RL32 pad 1: Net-(LED32-PadA) -> Net-(LED49-PadA)
- SW80 pad 1: Col9 -> Col11
- U1 pad 16: Net-(U1-Pad16) -> LED_PWM
- U1 pad 28: Net-(U1-Pad28) -> RGB_3V3
Routing:
- net Net-(Q2-Pad1): track 552.3 -> 1655.8 mm, vias 0 -> 2
- net 5V: track 158.8 -> 571.5 mm, vias 0 -> 2
- net Row5: track 0.00 -> 283.6 mm
- net Row4: track 0.00 -> 270.5 mm, vias 0 -> 2
- net Net-(U1-Pad16): track 205.8 -> 0.00 mm
- net Col1: track 21.8 -> 167.9 mm
- net Col2: track 0.00 -> 137.8 mm
- net Col3: track 0.00 -> 112.8 mm
- net Col7: track 0.00 -> 108.4 mm
- net Col11: track 0.00 -> 99.0 mm
- net Net-(U1-Pad21): track 126.7 -> 38.1 mm
- net LED_PWM: track 0.00 -> 79.1 mm, vias 0 -> 2
- net Col4: track 0.00 -> 71.9 mm
- net Col9: track 0.00 -> 71.0 mm
- net Col6: track 0.00 -> 71.0 mm
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Other:
- board text removed: "P20"
- board text removed: "P21"
- board text removed: "P22"
- board text removed: "P25"
- board text removed: "P26"
- board text removed: "P27"
- board text removed: "P28"
- board text removed: "P29"
- board text removed: "P30"
- board text removed: "P31"
- board text removed: "P38"
- board text removed: "P39"
- board text removed: "P40"
- board text removed: "P41"

Commit message: Assign col and row pins
Parts:
- removed DSH1: RB060M-60TR, acheron_Components:D_SOD-123
- added SW48: N, acheron_MX_SolderMask:MX100, F.Cu at (208.1, 148.5)
- moved D67 0.51 mm to (112.9, 138.2)
Connections:
- CSH2 pad 2: Net-(CSH2-Pad2) -> CASE
- D62 pad 2: Net-(D62-Pad2) -> L9
- RSH2 pad 1: Net-(CSH2-Pad2) -> CASE
- SW62 pad 2: Net-(D62-Pad2) -> L9
- U1 pad 10: Net-(U1-Pad10) -> Col4
- U1 pad 11: Net-(U1-Pad11) -> Col3
- U1 pad 12: Net-(U1-Pad12) -> Col2
- U1 pad 13: Net-(U1-Pad13) -> Row3
- U1 pad 14: Net-(U1-Pad14) -> Col14
- U1 pad 15: Net-(U1-Pad15) -> Col13
- U1 pad 17: Net-(U1-Pad17) -> Col12
- U1 pad 18: Net-(U1-Pad18) -> Col11
- U1 pad 19: Net-(U1-Pad19) -> Col10
- U1 pad 2: Net-(U1-Pad2) -> Row2
- U1 pad 20: Net-(U1-Pad20) -> Col9
- U1 pad 21: Net-(U1-Pad21) -> Row4
- U1 pad 22: Net-(U1-Pad22) -> Row5
- U1 pad 3: Net-(U1-Pad3) -> Col8
- U1 pad 4: Net-(U1-Pad4) -> Col7
- U1 pad 46: Net-(U1-Pad46) -> Row1
- U1 pad 5: Net-(U1-Pad5) -> Col6
- U1 pad 6: Net-(U1-Pad6) -> Col5
Routing:
- net Net-(U1-Pad14): track 251.0 -> 0.00 mm
- net Net-(U1-Pad15): track 241.7 -> 0.00 mm
- net Col14: track 166.8 -> 404.3 mm
- net Net-(U1-Pad13): track 231.4 -> 0.00 mm
- net Col13: track 179.2 -> 407.9 mm
- net Col12: track 102.5 -> 311.0 mm
- net Col11: track 99.0 -> 292.2 mm
- net Net-(U1-Pad17): track 187.5 -> 0.00 mm
- net Col10: track 71.0 -> 249.7 mm
- net Net-(U1-Pad18): track 169.5 -> 0.00 mm
- net Col9: track 71.0 -> 224.0 mm
- net Net-(U1-Pad19): track 150.5 -> 0.00 mm
- net Net-(U1-Pad20): track 132.0 -> 0.00 mm
- net Col8: track 71.0 -> 201.5 mm
- net Col7: track 108.4 -> 218.8 mm
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
Commit message: Run DRC, finish pin assignment
Parts:
- removed L9: Warning, acheron_Graphics:warning_sign_3.6x3.2mm
- added CR3: 100n, Capacitor_SMD:C_0805_2012Metric, F.Cu at (88.5, 140.4)
- added CR4: 100n, Capacitor_SMD:C_0805_2012Metric, F.Cu at (88.5, 137.5)
- added D60: 1N4148, acheron_Components:D_SOD-123, F.Cu at (92.6, 160.4)
- added ROT1: Rotary_Encoder_Switch, acheron_Hardware:ALPS_EC11E, F.Cu at (80.7, 148.5)
- added RR2: 10k, acheron_Components:R_SMD_1206, F.Cu at (97.9, 140.4)
- added RR3: 10k, acheron_Components:R_SMD_1206, F.Cu at (92.8, 140.4)
- added RR4: 10k, acheron_Components:R_SMD_1206, F.Cu at (97.9, 137.5)
- added RR5: 10k, acheron_Components:R_SMD_1206, F.Cu at (92.8, 137.5)
- J2: value Conn_01x14 -> Conn_01x12; footprint acheron_Connectors:PinHeader_1x14_P2.54mm_Vertical -> acheron_Connectors:PinHeader_1x12_P2.54mm_Vertical
- moved SW61 32.1 mm to (80.7, 148.5)
- moved SW62 20.2 mm to (106.9, 148.5)
- moved L1 19.1 mm to (248.9, 186.3)
- moved L4 19.1 mm to (247.4, 186.6)
- moved RL60 8.87 mm to (75.3, 158.0), turned to 270 degrees
- moved L5 7.04 mm to (84.0, 137.8)
- moved LED62 5.95 mm to (80.7, 153.6)
- moved LED60 5.95 mm to (106.9, 153.6)
Connections:
- D62 pad 2: L9 -> ROT_S1
- RGUI_125 pad 1: Col12 -> Col11
- SW58 pad 1: Col12 -> Col11
- SW59 pad 2: Col13 -> Col12
- SW60 pad 1: Col14 -> Col13
- SW61 pad 1: Col13 -> Col14
- SW61 pad 2: Net-(D53-Pad2) -> ROT_S1
- SW62 pad 1: Col14 -> Col13
- SW62 pad 2: L9 -> Net-(D53-Pad2)
- SW80 pad 1: Col11 -> Col10
- SW81 pad 1: Col12 -> Col11
- SW83 pad 1: Col13 -> Col12
- SW84 pad 1: Col13 -> Col12
- SW86 pad 1: Col14 -> Col13
- U1 pad 26: Net-(U1-Pad26) -> Extra12
- U1 pad 27: Net-(U1-Pad27) -> Extra11
- U1 pad 29: Net-(U1-Pad29) -> Extra10
- U1 pad 30: Net-(U1-Pad30) -> Extra9
- U1 pad 31: Net-(U1-Pad31) -> Extra8
- U1 pad 38: Net-(U1-Pad38) -> Extra7
- U1 pad 39: Net-(U1-Pad39) -> Extra6
- U1 pad 40: Net-(U1-Pad40) -> Extra5
- U1 pad 41: Net-(U1-Pad41) -> Extra4
- U1 pad 42: Net-(U1-Pad42) -> Extra3
- U1 pad 43: Net-(U1-Pad43) -> Extra2
- U1 pad 45: Net-(U1-Pad45) -> Extra1
Routing:
- net ENC_B: track 0.00 -> 305.1 mm, vias 0 -> 1
- net ENC_A: track 0.00 -> 301.8 mm, vias 0 -> 1
- net 3.3V: track 320.2 -> 464.3 mm, vias 7 -> 8
- net Extra1: track 0.00 -> 47.9 mm
- net Net-(U1-Pad45): track 45.7 -> 0.00 mm
- net Extra2: track 0.00 -> 43.5 mm
- net Net-(U1-Pad43): track 42.1 -> 0.00 mm
- net Extra3: track 0.00 -> 39.4 mm
- net Net-(U1-Pad42): track 37.9 -> 0.00 mm
- net Extra4: track 0.00 -> 36.7 mm
- net Net-(U1-Pad41): track 35.3 -> 0.00 mm
- net Extra5: track 0.00 -> 34.0 mm
- net Net-(U1-Pad40): track 32.9 -> 0.00 mm
- net Extra6: track 0.00 -> 31.3 mm
- net Col10: track 249.7 -> 280.3 mm
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Other:
- board text added: "A10"
- board text added: "A2"
- board text added: "A8"
- board text added: "A9"
- board text added: "B13"
- board text added: "B15"
- board text added: "B3"
- board text added: "B4"
- board text added: "B5"
- board text added: "B6"
- board text added: "B7"
- board text added: "B8"
