File: kicadFiles/tsuki.sch (KiCad schematic (older format))
At the start: 392 parts, among them J1 TYPE-C-31-M12_13, J2 Conn_01x12, J3 Conn_ARM_JTAG_SWD_10, Q1 BSS138, Q2 AO4407A, SW1 ESC, SW10 9, SW11 0, SW12 -_, SW13 +=, SW14 2U BKSP, SW15 TAB_150, SW16 Q, SW17 W, SW18 E, SW19 R, SW2 1, SW20 T, SW21 Y, SW22 U, SW23 I, SW24 O, SW25 P, SW26 [{, SW27 ]}, SW28 \\|_150, SW29 CAPS_175, SW3 2, SW30 A, SW31 S, SW32 D, SW33 F, SW34 G, SW35 H, SW36 J, SW37 K, SW38 L, SW39 :;, SW4 3, SW40 \"', SW41 ENTER_225, SW42 LSHIFT_225, SW43 Z, SW44 X, SW45 C, SW46 V, SW47 B, SW48 N, SW49 M, SW5 4, SW50 <,, SW51 >., SW52 ?/, SW53 RSHIFT_275, SW54 LCTRL_150, SW55 LGUI_100, SW56 LALT_150, SW58 RALT_150, SW59 RGUI_150, SW6 5, SW60 RCTRL_150, SW61 FN_100, SW62 RSHIFT_175, SW63 STEPPED_CAPS_125, SW64 1U LBKSP, SW65 1U RBKSP, SW66 ISO_100, SW67 ISO_ENTER, SW68 LCTRL_125, SW69 LGUI_125, SW7 6, SW70 LGUI_100, SW71 LALT_125, SW72 LALT_150, SW75 SPACE_625, SW77 SPACE_700, SW8 7, SW80 RALT_125, SW81 RALT_150, SW83 RGUI_125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

Commit message: Adjusted schematic
Parts:
- removed D66: 1N4148, acheron_Components:D_SOD-123, symbol Device:D
- removed LED67, LED70: LED, acheron_Components:LED_THT_2.54mm, symbol tsuki-rescue:LED-acheronSymbols
- removed RL68: 420R, acheron_Components:R_SMD_1206, symbol Device:R_Small
- removed SW55: LGUI_100, acheron_MX_SolderMask:MX150, symbol tsuki-rescue:MXSwitch-acheronSymbols
- removed SW56: LALT_150, acheron_MX_SolderMask:MX150, symbol tsuki-rescue:MXSwitch-acheronSymbols
- added D63: 1N4148, acheron_Components:D_SOD-123, symbol Device:D
- SW59: value RGUI_150 -> RGUI_100; footprint acheron_MX_SolderMask:MX150 -> acheron_MX_SolderMask:MX100
Connections:
- net Col10: now also SW58.1 (Col)
- net Col11: now also SW59.1 (Col); no longer SW58.1 (Col)
- net Col12: no longer SW59.2 (Row)
- net L6: now also D58.2 (A), SW58.2 (Row)
- net L7: now also D59.2 (A), SW59.2 (Row); no longer D58.2 (A), SW58.2 (Row)
- net L8: now also D63.2 (A); no longer D59.2 (A), SW59.1 (Col)
- net Row5: now also D63.1 (K)
- net at LED78.A, LED79.A, RL75.1: no longer LED77.A
- net at LED75.A, LED76.A, RL73.1: now also LED77.A
Other:
- note added: "Encoder"
- note added: "Per-keys LEDs"
- note added: "RGB Underglow"
- moved on the sheet: CB1, CB2, CB3, CB4, CB5, CB6, CB7, CB8, CR1, CR2, CR3, CR4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

Commit message: Further adjust schematic
Connections:
- net L2: now also D56.2 (A), SW71.2 (Row)
- net L3: no longer D56.2 (A), SW71.2 (Row)
Other:
- note added: "Warning\nsigns"
- moved on the sheet: D55, D56, L5, L6, L7, L8

Commit message: Refresh KLE, finish PCB and schematic
Parts:
- J2: footprint acheron_Connectors:PinHeader_1x12_P2.54mm_Vertical -> acheron_Connectors:PinHeader_1x10_P2.54mm_Vertical; symbol Connector_Generic:Conn_01x12 -> Connector_Generic:Conn_01x10
- renumbered CB8 to CB1, CB7 to CB2, CB1 to CB5, CB2 to CB6, CB5 to CB7, CB6 to CB8, CR3 to CR1, CR4 to CR2, CR2 to CR3, CR1 to CR4, CSH2 to CSH1, CSH1 to CSH2, D65 to D28, D28 to D41, D41 to D42, D42 to D43, D61 to D44, D43 to D45, D44 to D46, D45 to D47, D46 to D48, D47 to D49, D48 to D50, D49 to D51, D50 to D52, D51 to D53, D52 to D54, D53 to D55, D67 to D56, D54 to D57, D57 to D58, D58 to D59, D59 to D60, D62 to D61, D63 to D62, D55 to D63, D56 to D64, D60 to D65, J3 to J1, J1 to J3, L2 to L1, L5 to L2, L6 to L3, L1 to L4, L7 to L5, L3 to L6, L8 to L7, L4 to L8, L10 to L9, LED68 to LED67, LED69 to LED68, LED71 to LED69, LED72 to LED70, LED73 to LED71, LED74 to LED72, LED77 to LED73, LED76 to LED74, LED78 to LED76, LED79 to LED77, LED80 to LED78, LED81 to LED79, Q2 to QLED1, QRST2 to QLED2, RCC2 to RCC1, RCC1 to RCC2, RL16 to RL15, RL17 to RL16, RL18 to RL17, RL19 to RL18, RL20 to RL19, RL21 to RL20, RL22 to RL21, RL23 to RL22, RL24 to RL23, RL25 to RL24, RL26 to RL25, RL27 to RL26, RL28 to RL27, RL29 to RL28, RL30 to RL29, RL31 to RL30, RL15 to RL31, RL33 to RL32, RL34 to RL33, RL35 to RL34, RL36 to RL35, RL37 to RL36, RL38 to RL37, RL39 to RL38, RL40 to RL39, RL41 to RL40, RL42 to RL41, RL43 to RL42, RL44 to RL43, RL45 to RL44, RL46 to RL45, RL32 to RL46, RL48 to RL47, RL49 to RL48, RL50 to RL49, RL51 to RL50, RL52 to RL51, RL53 to RL52, RL54 to RL53, RL55 to RL54, RL56 to RL55, RL57 to RL56, RL58 to RL57, RL60 to RL58, RL61 to RL59, RL63 to RL60, RL66 to RL61, RL69 to RL62, RL71 to RL63, RL73 to RL64, RL75 to RL65, RL77 to RL66, RLED3 to RLED2, RLED2 to RLED3, RR2 to RR1, RR4 to RR2, RR5 to RR4, RR1 to RR5, RS2 to RS1, RS1 to RS2, RSH2 to RSH1, RSH1 to RSH2, SW64 to SW1, SW9 to SW10, SW10 to SW11, SW11 to SW12, SW12 to SW13, SW13 to SW14, SW14 to SW15, SW15 to SW16, SW16 to SW17, SW17 to SW18, SW18 to SW19, SW1 to SW2, SW19 to SW20, SW20 to SW21, SW21 to SW22, SW22 to SW23, SW23 to SW24, SW24 to SW25, SW25 to SW26, SW26 to SW27, SW27 to SW28, SW65 to SW29, SW2 to SW3, SW63 to SW30, SW29 to SW31, SW30 to SW32, SW31 to SW33, SW32 to SW34, SW33 to SW35, SW34 to SW36, SW35 to SW37, SW36 to SW38, SW37 to SW39, SW3 to SW4, SW38 to SW40, SW39 to SW41, SW40 to SW42, SW28 to SW43, SW41 to SW44, SW67 to SW45, SW62 to SW46, SW42 to SW47, SW66 to SW48, SW43 to SW49, SW4 to SW5, SW44 to SW50, SW45 to SW51, SW46 to SW52, SW47 to SW53, SW48 to SW54, SW49 to SW55, SW50 to SW56, SW51 to SW57, SW52 to SW58, SW53 to SW59, SW5 to SW6, SW88 to SW60, SW89 to SW61, SW54 to SW62, SW58 to SW63, SW59 to SW64, SW61 to SW65, SW68 to SW66, SW69 to SW67, SW71 to SW68, SW75 to SW69, SW6 to SW7, SW80 to SW70, RGUI_125 to SW71, SW83 to SW72, SW86 to SW73, SW70 to SW74, SW72 to SW75, SW77 to SW76, SW81 to SW77, SW84 to SW78, SW60 to SW79, SW7 to SW8, SW8 to SW9, U2 to U1, U1 to U2
Connections:
- net Extra1 is gone; now on net Extra3: J2.1 (Pin_1)
- net Extra10: now also J2.8 (Pin_8); no longer J2.10 (Pin_10)
- net Extra11: now also J2.9 (Pin_9); no longer J2.11 (Pin_11)
- net Extra12: now also J2.10 (Pin_10); no longer J2.12 (Pin_12)
- net Extra2: no longer J2.2 (Pin_2)
- net Extra3: no longer J2.3 (Pin_3)
- net Extra4: now also J2.2 (Pin_2); no longer J2.4 (Pin_4)
- net Extra5: now also J2.3 (Pin_3); no longer J2.5 (Pin_5)
- net Extra6: now also J2.4 (Pin_4); no longer J2.6 (Pin_6)
- net Extra7: now also J2.5 (Pin_5); no longer J2.7 (Pin_7)
- net Extra8: now also J2.6 (Pin_6); no longer J2.8 (Pin_8)
- net Extra9: now also J2.7 (Pin_7); no longer J2.9 (Pin_9)
