File: kicadFiles/tsuki.sch (KiCad schematic (older format))
At the start: 387 parts, among them J1 Conn_ARM_JTAG_SWD_10, J2 Conn_01x12, J3 TYPE-C-31-M12_13, Q1 BSS138, SW1 1U LBKSP, SW10 8, SW11 9, SW12 0, SW13 -_, SW14 +=, SW15 2U BKSP, SW16 TAB_150, SW17 Q, SW18 W, SW19 E, SW2 ESC, SW20 R, SW21 T, SW22 Y, SW23 U, SW24 I, SW25 O, SW26 P, SW27 [{, SW28 ]}, SW29 1U RBKSP, SW3 1, SW30 STEPPED_CAPS_125, SW31 CAPS_175, SW32 A, SW33 S, SW34 D, SW35 F, SW36 G, SW37 H, SW38 J, SW39 K, SW4 2, SW40 L, SW41 :;, SW42 \"', SW43 \\|_150, SW44 ENTER_225, SW45 ISO_ENTER, SW46 RSHIFT_175, SW47 LSHIFT_225, SW48 ISO_100, SW49 Z, SW5 3, SW50 X, SW51 C, SW52 V, SW53 B, SW54 N, SW55 M, SW56 <,, SW57 >., SW58 ?/, SW59 RSHIFT_275, SW6 4, SW60 ISO_\\_100, SW61 LSHIFT_125, SW62 LCTRL_150, SW63 RALT_150, SW64 RGUI_100, SW65 FN_100, SW66 LCTRL_125, SW67 LGUI_125, SW68 LALT_125, SW69 SPACE_625, SW7 5, SW70 RALT_125, SW71 FN_125, SW72 RGUI_125, SW73 RCTRL_125, SW74 LGUI_100, SW75 LALT_150, SW76 SPACE_700, SW77 RALT_150, SW78 RGUI_100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

Commit message: Final preparations for release pre-Alpha
Connections:
- net L2: no longer D64.2 (A), SW68.2 (Row)
- net L3: now also D64.2 (A), SW68.2 (Row)
Changed lines of the file:
@@
 Connection ~ 17500 7150
 Text GLabel 18575 7150 2    50   Input ~ 0
-L2
+L3
 Wire Wire Line
 	18575 7150 18500 7150
